File: KiCad/LED Panel.kicad_pcb (KiCad board)
At the start: 2 copper layers, 5 parts, among them J1 Conn_01x05_Male, SW1 SW_Push, SW2 SW_Push, SW3 SW_Push, SW4 SW_Push

Commit message: Update electronic model
Parts:
- moved SW1 47.1 mm to (184.3, 110.6)
- moved SW4 24.1 mm to (184.2, 86.4)
- moved SW3 23.1 mm to (164.0, 99.1)
- moved SW2 22.9 mm to (143.7, 86.4)
Connections:
- J1 pad 1: GND -> Net-(J1-Pad1)
- J1 pad 5: Net-(J1-Pad5) -> GND
- SW1 pad 1: Net-(J1-Pad2) -> Net-(J1-Pad1)
- SW2 pad 2: Net-(J1-Pad3) -> Net-(J1-Pad2)
- SW3 pad 1: Net-(J1-Pad4) -> Net-(J1-Pad3)
- SW4 pad 2: Net-(J1-Pad5) -> Net-(J1-Pad4)
Routing:
- net GND: track 93.7 -> 0.25 mm
- net Net-(J1-Pad1): track 0.00 -> 52.8 mm
- net Net-(J1-Pad5): track 50.0 -> 0.00 mm
- net Net-(J1-Pad3): track 16.9 -> 28.6 mm
- net Net-(J1-Pad4): track 56.6 -> 50.1 mm
- net Net-(J1-Pad2): track 31.4 -> 25.5 mm
- added copper zone on F.Cu, net GND
