File: KiCad/LED Panel.sch (KiCad schematic (older format))
At the start: 5 parts, among them J1 Conn_01x05_Male, SW1 SW_Push, SW2 SW_Push, SW3 SW_Push, SW4 SW_Push

Commit message: Update electronic model
Connections:
- net GND: now also J1.5 (Pin_5); no longer J1.1 (Pin_1)
- net at SW1.1: now also J1.1 (Pin_1); no longer J1.2 (Pin_2)
- net at SW2.2: now also J1.2 (Pin_2); no longer J1.3 (Pin_3)
- net at SW3.1: now also J1.3 (Pin_3); no longer J1.4 (Pin_4)
- net at SW4.2: now also J1.4 (Pin_4); no longer J1.5 (Pin_5)
Changed lines of the file:
@@
 EESchema Schematic File Version 4
+LIBS:LED Panel-cache
 EELAYER 26 0
 EELAYER END
@@
 F 1 "SW_Push" H 5350 2394 50  0000 C CNN
 F 2 "Button_Switch_THT:SW_PUSH-12mm_Wuerth-430476085716" H 5350 2400 50  0001 C CNN
-F 3 "" H 5350 2400 50  0001 C CNN
+F 3 "UP button" H 5350 2400 50  0001 C CNN
 	1    5350 2200
 	1    0    0    -1
@@
 F 1 "SW_Push" H 5350 2944 50  0000 C CNN
 F 2 "Button_Switch_THT:SW_PUSH-12mm_Wuerth-430476085716" H 5350 2950 50  0001 C CNN
-F 3 "" H 5350 2950 50  0001 C CNN
+F 3 "BACK button" H 5350 2950 50  0001 C CNN
 	1    5350 2750
 	1    0    0    -1
@@
 F 1 "SW_Push" H 6150 2394 50  0000 C CNN
 F 2 "Button_Switch_THT:SW_PUSH-12mm_Wuerth-430476085716" H 6150 2400 50  0001 C CNN
-F 3 "" H 6150 2400 50  0001 C CNN
+F 3 "OK button" H 6150 2400 50  0001 C CNN
 	1    6150 2200
 	1    0    0    -1
@@
 F 1 "SW_Push" H 6150 2944 50  0000 C CNN
 F 2 "Button_Switch_THT:SW_PUSH-12mm_Wuerth-430476085716" H 6150 2950 50  0001 C CNN
-F 3 "" H 6150 2950 50  0001 C CNN
+F 3 "DOWN button" H 6150 2950 50  0001 C CNN
 	1    6150 2750
 	1    0    0    -1
@@
 	5750 2750 5950 2750
 Wire Wire Line
-	4450 2400 5150 2400
-Wire Wire Line
-	5150 2400 5150 2200
-Wire Wire Line
-	4450 2500 5200 2500
-Wire Wire Line
-	4450 2600 5150 2600
-Wire Wire Line
 	5150 2600 5150 2750
 Wire Wire Line
-	4450 2850 6350 2850
-Wire Wire Line
 	6350 2750 6350 2850
-Wire Wire Line
-	4450 2850 4450 2700
 Wire Wire Line
 	5750 2200 5750 2750
@@
 Wire Wire Line
 	5750 1750 5050 1750
-Wire Wire Line
-	4700 1750 4700 2300
-Wire Wire Line
-	4700 2300 4450 2300
-Wire Wire Line
-	5200 2500 5200 2350
-Wire Wire Line
-	5200 2350 6350 2350
 Wire Wire Line
 	6350 2200 6350 2350
@@
 Connection ~ 5050 1750
 Wire Wire Line
-	5050 1750 4700 1750
+	4000 1750 4000 2800
+Wire Wire Line
+	4000 2800 4450 2800
+Wire Wire Line
+	4450 2800 4450 2700
+Wire Wire Line
+	4000 1750 5050 1750
+Wire Wire Line
+	5150 2200 4850 2200
+Wire Wire Line
+	4850 2200 4850 2300
+Wire Wire Line
+	4850 2300 4450 2300
+Wire Wire Line
+	4850 2350 4850 2400
+Wire Wire Line
+	4850 2400 4450 2400
+Wire Wire Line
+	4850 2350 6350 2350
+Wire Wire Line
+	5150 2600 4850 2600
+Wire Wire Line
+	4850 2600 4850 2500
+Wire Wire Line
+	4850 2500 4450 2500
+Wire Wire Line
+	6350 2850 4750 2850
+Wire Wire Line
+	4750 2850 4750 2600
+Wire Wire Line
+	4750 2600 4450 2600
 $EndSCHEMATC
